Commit message: Add form-locking pizza serving demo

File: isaacpjt/M0609/doosan-robot2/urdf/m0609_moveit.urdf.xacro (robot description, xacro)
@@ -250,14 +250,12 @@
 			<child link="tool0"/>
 		</joint>
-		<!-- Detailed OnRobot RG2 model. The fingers use the zero-angle pose for
-		     the current six-axis arm test; Isaac Sim retains the live gripper
-		     articulation. The fixed links keep RViz and MoveIt state complete. -->
+		<!-- Detailed OnRobot RG2 model. rg2_finger_joint is the actuated joint;
+		     the remaining linkage joints follow it through URDF mimic tags. -->
 		<material name="rg2_silver"><color rgba="0.68 0.69 0.68 1"/></material>
 		<material name="rg2_blue"><color rgba="0.216 0.592 0.812 1"/></material>
 		<xacro:macro name="rg2_mesh_link" params="name mesh visual_xyz:='0 0 0' color:='rg2_silver'">
 			<link name="${name}">
-				<!-- Fixed RG2 parts still become individual rigid bodies when
-				     Isaac's importer preserves fixed joints.  Give them finite
-				     mass properties to avoid negative-mass fallback and jitter. -->
+				<!-- Every imported RG2 link needs finite mass properties for a
+				     stable PhysX articulation. -->
 				<inertial>
 					<origin xyz="0 0 0" rpy="0 0 0"/>
@@ -305,33 +303,50 @@
 			<origin xyz="-0.02705 0 0.04445" rpy="0.0101229097 0 0"/>
 		</joint>
-		<joint name="rg2_left_inner_knuckle_joint" type="fixed">
+		<joint name="rg2_left_inner_knuckle_joint" type="revolute">
 			<parent link="rg2_base_link"/>
 			<child link="rg2_left_inner_knuckle"/>
 			<origin xyz="0.03455 -0.009367 0.092397" rpy="0 0.415388362 0"/>
-		</joint>
-		<joint name="rg2_finger_joint" type="fixed">
+			<axis xyz="0 0.999949 -0.010122"/>
+			<limit effort="50" lower="-1.19" upper="0.01" velocity="2"/>
+			<mimic joint="rg2_finger_joint" multiplier="-1" offset="0"/>
+		</joint>
+		<joint name="rg2_finger_joint" type="revolute">
 			<parent link="rg2_base_link"/>
 			<child link="rg2_right_outer_knuckle"/>
 			<origin xyz="0.01005 -0.009534 0.075898" rpy="0 -0.415388362 0"/>
-		</joint>
-		<joint name="rg2_left_outer_knuckle_joint" type="fixed">
+			<axis xyz="0 0.999949 -0.010122"/>
+			<limit effort="50" lower="0" upper="1.18" velocity="2"/>
+		</joint>
+		<joint name="rg2_left_outer_knuckle_joint" type="revolute">
 			<parent link="rg2_base_link"/>
 			<child link="rg2_left_outer_knuckle"/>
 			<origin xyz="0.04405 -0.009534 0.075898" rpy="0 0.415388362 0"/>
-		</joint>
-		<joint name="rg2_left_inner_finger_joint" type="fixed">
+			<axis xyz="0 0.999949 -0.010122"/>
+			<limit effort="50" lower="-1.19" upper="0.01" velocity="2"/>
+			<mimic joint="rg2_finger_joint" multiplier="-1" offset="0"/>
+		</joint>
+		<joint name="rg2_left_inner_finger_joint" type="revolute">
 			<parent link="rg2_left_outer_knuckle"/>
 			<child link="rg2_left_inner_finger"/>
 			<origin xyz="0.039748 0.004784 0.037968" rpy="0 -0.415388362 0"/>
-		</joint>
-		<joint name="rg2_right_inner_finger_joint" type="fixed">
+			<axis xyz="0 -0.999949 0.010122"/>
+			<limit effort="50" lower="-1.19" upper="0.01" velocity="2"/>
+			<mimic joint="rg2_finger_joint" multiplier="-1" offset="0"/>
+		</joint>
+		<joint name="rg2_right_inner_finger_joint" type="revolute">
 			<parent link="rg2_right_outer_knuckle"/>
 			<child link="rg2_right_inner_finger"/>
 			<origin xyz="-0.039748 0.004784 0.037968" rpy="0 0.415388362 0"/>
-		</joint>
-		<joint name="rg2_right_inner_knuckle_joint" type="fixed">
+			<axis xyz="0 0.999949 -0.010122"/>
+			<limit effort="50" lower="-1.19" upper="0.01" velocity="2"/>
+			<mimic joint="rg2_finger_joint" multiplier="-1" offset="0"/>
+		</joint>
+		<joint name="rg2_right_inner_knuckle_joint" type="revolute">
 			<parent link="rg2_base_link"/>
 			<child link="rg2_right_inner_knuckle"/>
 			<origin xyz="0.01955 -0.009367 0.092397" rpy="0 -0.415388362 0"/>
+			<axis xyz="0 0.999949 -0.010122"/>
+			<limit effort="50" lower="-0.01" upper="1.19" velocity="2"/>
+			<mimic joint="rg2_finger_joint" multiplier="1" offset="0"/>
 		</joint>
 		<link name="rg2_tcp"/>

File: src/ridgeback_m0609_description/urdf/ridgeback_m0609.urdf (robot description, URDF)
Before this commit: robot ridgeback_m0609, 27 links, 26 joints
Links:
- link serving_shelf_link: geometry collision box size=0.025 0.58 0.54; collision box size=0.035 0.035 0.56
Joints:
- joint rg2_finger_joint: axis (none) -> 0 0.999949 -0.010122; limit (none) -> lower=0 upper=1.18 effort=50 velocity=2; type fixed -> revolute
- joint rg2_left_inner_finger_joint: axis (none) -> 0 -0.999949 0.010122; limit (none) -> lower=-1.19 upper=0.01 effort=50 velocity=2; mimic (none) -> joint=rg2_finger_joint multiplier=-1 offset=0; type fixed -> revolute
- joint rg2_left_inner_knuckle_joint: axis (none) -> 0 0.999949 -0.010122; limit (none) -> lower=-1.19 upper=0.01 effort=50 velocity=2; mimic (none) -> joint=rg2_finger_joint multiplier=-1 offset=0; type fixed -> revolute
- joint rg2_left_outer_knuckle_joint: axis (none) -> 0 0.999949 -0.010122; limit (none) -> lower=-1.19 upper=0.01 effort=50 velocity=2; mimic (none) -> joint=rg2_finger_joint multiplier=-1 offset=0; type fixed -> revolute
- joint rg2_right_inner_finger_joint: axis (none) -> 0 0.999949 -0.010122; limit (none) -> lower=-1.19 upper=0.01 effort=50 velocity=2; mimic (none) -> joint=rg2_finger_joint multiplier=-1 offset=0; type fixed -> revolute
- joint rg2_right_inner_knuckle_joint: axis (none) -> 0 0.999949 -0.010122; limit (none) -> lower=-0.01 upper=1.19 effort=50 velocity=2; mimic (none) -> joint=rg2_finger_joint multiplier=1 offset=0; type fixed -> revolute

File: src/ridgeback_m0609_description/urdf/ridgeback_m0609.urdf.xacro (robot description, xacro)
@@ -109,12 +109,24 @@
       <geometry><box size="0.74 0.62 0.025"/></geometry>
     </collision>
+    <!-- Upper tray with a -X/+Y serving notch.  The rear panel and +X rail
+         remain, while the plate-side front edge is open for horizontal RG2
+         access. -->
     <visual>
-      <origin xyz="0 0 0.64"/>
-      <geometry><box size="0.74 0.62 0.025"/></geometry>
+      <origin xyz="0 -0.145 0.64"/>
+      <geometry><box size="0.74 0.33 0.025"/></geometry>
       <material name="shelf_tray"/>
     </visual>
     <collision>
-      <origin xyz="0 0 0.64"/>
-      <geometry><box size="0.74 0.62 0.025"/></geometry>
+      <origin xyz="0 -0.145 0.64"/>
+      <geometry><box size="0.74 0.33 0.025"/></geometry>
+    </collision>
+    <visual>
+      <origin xyz="0.21 0.165 0.64"/>
+      <geometry><box size="0.32 0.29 0.025"/></geometry>
+      <material name="shelf_tray"/>
+    </visual>
+    <collision>
+      <origin xyz="0.21 0.165 0.64"/>
+      <geometry><box size="0.32 0.29 0.025"/></geometry>
     </collision>
     <visual>
