Commit message: 로봇팔 전방 배치 및 복도 방향 서빙 동작 수정

File: serving_robot/src/ridgeback_m0609_description/urdf/ridgeback_m0609.urdf (robot description, URDF)
Before this commit: robot ridgeback_m0609, 27 links, 26 joints
Joints:
- joint arm_mount_joint: origin xyz=-0.22 0 0.875 -> xyz=0.22 0 0.875

File: serving_robot/src/ridgeback_m0609_description/urdf/ridgeback_m0609.urdf.xacro (robot description, xacro)
@@ -97,6 +97,7 @@
   <xacro:ridgeback_wheel prefix="rear_left"   x="${-wheel_x}" y="${ wheel_y}"/>
   <xacro:ridgeback_wheel prefix="rear_right"  x="${-wheel_x}" y="${-wheel_y}"/>
-  <!-- Fixed stainless shelf.  Two food trays are below the arm plate, and the
-       arm is offset rearward so it can reach both trays and the table. -->
+  <!-- Fixed stainless shelf.  The arm is offset toward base +X so Nav2 can
+       approach a service table forwards; the asymmetric tray details are
+       mirrored so the pizza remains behind the arm during transport. -->
   <link name="serving_shelf_link">
     <visual>
@@ -109,7 +110,6 @@
       <geometry><box size="0.74 0.62 0.025"/></geometry>
     </collision>
-    <!-- Upper tray with a -X/+Y serving notch.  The rear panel and +X rail
-         remain, while the plate-side front edge is open for horizontal RG2
-         access. -->
+    <!-- Mirrored upper tray: retain the +X-facing service layout while the
+         plate-side -X edge remains open for RG2 access from the front arm. -->
     <visual>
       <origin xyz="0 -0.145 0.64"/>
@@ -122,10 +122,10 @@
     </collision>
     <visual>
-      <origin xyz="0.21 0.165 0.64"/>
+      <origin xyz="-0.21 0.165 0.64"/>
       <geometry><box size="0.32 0.29 0.025"/></geometry>
       <material name="shelf_tray"/>
     </visual>
     <collision>
-      <origin xyz="0.21 0.165 0.64"/>
+      <origin xyz="-0.21 0.165 0.64"/>
       <geometry><box size="0.32 0.29 0.025"/></geometry>
     </collision>
@@ -155,14 +155,14 @@
     <xacro:shelf_post x="-0.34" y="-0.28"/>
     <visual>
-      <origin xyz="-0.355 0 0.56"/>
+      <origin xyz="0.355 0 0.56"/>
       <geometry><box size="0.025 0.58 0.54"/></geometry>
       <material name="shelf_steel"/>
     </visual>
     <collision>
-      <origin xyz="-0.355 0 0.56"/>
+      <origin xyz="0.355 0 0.56"/>
       <geometry><box size="0.025 0.58 0.54"/></geometry>
     </collision>
     <inertial>
-      <origin xyz="-0.03 0 0.57"/>
+      <origin xyz="0.03 0 0.57"/>
       <mass value="20.0"/>
       <inertia ixx="1.20" ixy="0" ixz="0" iyy="1.25" iyz="0" izz="1.50"/>
@@ -188,5 +188,5 @@
     <parent link="serving_shelf_link"/>
     <child link="arm_mount_link"/>
-    <origin xyz="-0.22 0 0.875"/>
+    <origin xyz="0.22 0 0.875"/>
   </joint>
   <joint name="m0609_mount_joint" type="fixed">

Commit message: 서빙 트레이와 피자·음료·수저통 연속 배송 구현

File: serving_robot/src/ridgeback_m0609_description/urdf/ridgeback_m0609.urdf (robot description, URDF)
Before this commit: robot ridgeback_m0609, 27 links, 26 joints
Links:
- added link serving_tray_magnet_link, mass 0.02; visual cylinder length=0.002 radius=0.025
- added link upper_tray_left_link, mass 4.0; collision box size=0.015 0.285 0.045; collision box size=0.015 0.285 0.045
- added link upper_tray_right_link, mass 4.0; collision box size=0.015 0.285 0.045; collision box size=0.015 0.285 0.045
- link serving_shelf_link: geometry collision box size=0.025 0.58 0.54; collision box size=0.035 0.035 0.56
Joints:
- added joint serving_tray_magnet_joint: type fixed, parent serving_shelf_link, child serving_tray_magnet_link, origin xyz=-0.16 0 0.855 rpy=0 0 0
- added joint upper_tray_left_slide_joint: type prismatic, parent serving_shelf_link, child upper_tray_left_link, origin xyz=0 0.155 0.64, axis 0 1 0, limit lower=0.0 upper=0.25 effort=400 velocity=0.15
- added joint upper_tray_right_slide_joint: type prismatic, parent serving_shelf_link, child upper_tray_right_link, origin xyz=0 -0.155 0.64, axis 0 -1 0, limit lower=0.0 upper=0.25 effort=400 velocity=0.15

File: serving_robot/src/ridgeback_m0609_description/urdf/ridgeback_m0609.urdf.xacro (robot description, xacro)
@@ -11,4 +11,5 @@
   <material name="shelf_steel"><color rgba="0.55 0.60 0.64 1"/></material>
   <material name="shelf_tray"><color rgba="0.16 0.24 0.30 1"/></material>
+  <material name="magnet_dark"><color rgba="0.08 0.09 0.10 1"/></material>
   <!-- Ridgeback dimensions and wheel placement come from Clearpath's Humble
        R100 description.  The base frame is at floor level. -->
@@ -98,6 +99,7 @@
   <xacro:ridgeback_wheel prefix="rear_right"  x="${-wheel_x}" y="${-wheel_y}"/>
   <!-- Fixed stainless shelf.  The arm is offset toward base +X so Nav2 can
-       approach a service table forwards; the asymmetric tray details are
-       mirrored so the pizza remains behind the arm during transport. -->
+       approach a service table forwards.  The second deck uses two powered
+       linear trays which meet at the centre while driving and extend toward
+       both robot sides after docking. -->
   <link name="serving_shelf_link">
     <visual>
@@ -110,23 +112,22 @@
       <geometry><box size="0.74 0.62 0.025"/></geometry>
     </collision>
-    <!-- Mirrored upper tray: retain the +X-facing service layout while the
-         plate-side -X edge remains open for RG2 access from the front arm. -->
-    <visual>
-      <origin xyz="0 -0.145 0.64"/>
-      <geometry><box size="0.74 0.33 0.025"/></geometry>
-      <material name="shelf_tray"/>
-    </visual>
-    <collision>
-      <origin xyz="0 -0.145 0.64"/>
-      <geometry><box size="0.74 0.33 0.025"/></geometry>
-    </collision>
-    <visual>
-      <origin xyz="-0.21 0.165 0.64"/>
-      <geometry><box size="0.32 0.29 0.025"/></geometry>
-      <material name="shelf_tray"/>
-    </visual>
-    <collision>
-      <origin xyz="-0.21 0.165 0.64"/>
-      <geometry><box size="0.32 0.29 0.025"/></geometry>
+    <!-- Fixed guide rails below the sliding second-deck trays. -->
+    <visual>
+      <origin xyz="0 0.14 0.615"/>
+      <geometry><box size="0.70 0.025 0.025"/></geometry>
+      <material name="shelf_steel"/>
+    </visual>
+    <collision>
+      <origin xyz="0 0.14 0.615"/>
+      <geometry><box size="0.70 0.025 0.025"/></geometry>
+    </collision>
+    <visual>
+      <origin xyz="0 -0.14 0.615"/>
+      <geometry><box size="0.70 0.025 0.025"/></geometry>
+      <material name="shelf_steel"/>
+    </visual>
+    <collision>
+      <origin xyz="0 -0.14 0.615"/>
+      <geometry><box size="0.70 0.025 0.025"/></geometry>
     </collision>
     <visual>
@@ -174,4 +175,80 @@
     <origin xyz="0 0 0"/>
   </joint>
+  <!-- The two halves fill the former notched second deck when retracted.
+       Both joints use positive 0..0.25 m commands; their opposing axes make
+       the trays extend symmetrically toward robot left and right. -->
+  <xacro:macro name="sliding_upper_tray" params="side y axis_y">
+    <link name="upper_tray_${side}_link">
+      <visual>
+        <geometry><box size="0.74 0.30 0.025"/></geometry>
+        <material name="shelf_tray"/>
+      </visual>
+      <collision>
+        <geometry><box size="0.74 0.30 0.025"/></geometry>
+      </collision>
+      <!-- Shallow outer rim helps drinks remain on the tray without blocking
+           top-down access at the centre seam. -->
+      <visual>
+        <origin xyz="0 ${axis_y * 0.1425} 0.0225"/>
+        <geometry><box size="0.74 0.015 0.045"/></geometry>
+        <material name="shelf_steel"/>
+      </visual>
+      <collision>
+        <origin xyz="0 ${axis_y * 0.1425} 0.0225"/>
+        <geometry><box size="0.74 0.015 0.045"/></geometry>
+      </collision>
+      <visual>
+        <origin xyz="0.3625 0 0.0225"/>
+        <geometry><box size="0.015 0.285 0.045"/></geometry>
+        <material name="shelf_steel"/>
+      </visual>
+      <collision>
+        <origin xyz="0.3625 0 0.0225"/>
+        <geometry><box size="0.015 0.285 0.045"/></geometry>
+      </collision>
+      <visual>
+        <origin xyz="-0.3625 0 0.0225"/>
+        <geometry><box size="0.015 0.285 0.045"/></geometry>
+        <material name="shelf_steel"/>
+      </visual>
+      <collision>
+        <origin xyz="-0.3625 0 0.0225"/>
+        <geometry><box size="0.015 0.285 0.045"/></geometry>
+      </collision>
+      <inertial>
+        <mass value="4.0"/>
+        <inertia ixx="0.0302" ixy="0" ixz="0" iyy="0.1827" iyz="0" izz="0.2127"/>
+      </inertial>
+    </link>
+    <joint name="upper_tray_${side}_slide_joint" type="prismatic">
+      <parent link="serving_shelf_link"/>
+      <child link="upper_tray_${side}_link"/>
+      <origin xyz="0 ${y} 0.64"/>
+      <axis xyz="0 ${axis_y} 0"/>
+      <limit lower="0.0" upper="0.25" effort="400" velocity="0.15"/>
+      <dynamics damping="80.0" friction="5.0"/>
+    </joint>
+  </xacro:macro>
+  <xacro:sliding_upper_tray side="left"  y="0.155"  axis_y="1"/>
+  <xacro:sliding_upper_tray side="right" y="-0.155" axis_y="-1"/>
+  <!-- Weak permanent magnet embedded flush in the fixed top deck beneath the
+       pizza-board centre.  This is a robot fixture, so it belongs in the
+       robot description rather than being spawned by the pizza task.  It is
+       visual-only: the existing deck collider remains the contact surface. -->
+  <link name="serving_tray_magnet_link">
+    <visual>
+      <geometry><cylinder radius="0.025" length="0.002"/></geometry>
+      <material name="magnet_dark"/>
+    </visual>
+    <inertial>
+      <mass value="0.02"/>
+      <inertia ixx="0.000003" ixy="0" ixz="0" iyy="0.000003" iyz="0" izz="0.000006"/>
+    </inertial>
+  </link>
+  <joint name="serving_tray_magnet_joint" type="fixed">
+    <parent link="serving_shelf_link"/>
+    <child link="serving_tray_magnet_link"/>
+    <origin xyz="-0.16 0 0.855" rpy="0 0 0"/>
+  </joint>
   <link name="arm_mount_link">
     <visual>
