Commit message: fix(nav_robot5): rename robot frame to literal base_link
nav2_util::getCurrentPose() (used internally by bt_navigator) has a
hardcoded C++ default of "base_link" for its robot-frame argument, and
at least one stock behavior-tree call path hits that default instead of
reading our robot_base_frame param. With the project's prior frame name
(ridgeback_base_link, present before this branch), that lookup always
failed, so goThroughPoses/goToPose fell into endless spin/backup
recovery and eventually aborted. Renaming the frame to plain
"base_link" everywhere (URDF links, nav2_params.yaml, topic_bridge,
nav_bootstrap, rail_navigator, rail_mission) matches nav2's fallback;
per-robot isolation still holds because TF stays split by topic
(/robot1/tf vs /robot2/tf), not by frame name.

Co-Authored-By: Claude Sonnet 5 <noreply@anthropic.com>

File: nav_robot5/src/two_wheel_rails/urdf/two_wheel_robot_robot1.urdf (robot description, URDF)
Before this commit: robot nav5_two_wheel_robot1, 4 links, 3 joints
Links:
- removed link ridgeback_base_link
- added link base_link; visual box size=0.84 0.70 0.36
Joints:
- joint left_wheel_visual_joint: parent ridgeback_base_link -> base_link
- joint nav_lidar_fixed_joint: parent ridgeback_base_link -> base_link
- joint right_wheel_visual_joint: parent ridgeback_base_link -> base_link

File: nav_robot5/src/two_wheel_rails/urdf/two_wheel_robot_robot2.urdf (robot description, URDF)
Before this commit: robot nav5_two_wheel_robot2, 4 links, 3 joints
Links:
- removed link ridgeback_base_link
- added link base_link; visual box size=0.84 0.70 0.36
Joints:
- joint left_wheel_visual_joint: parent ridgeback_base_link -> base_link
- joint nav_lidar_fixed_joint: parent ridgeback_base_link -> base_link
- joint right_wheel_visual_joint: parent ridgeback_base_link -> base_link
